Commit message: амтоматически генерируется новый пакет под ros/ros2

File: config/solid3_description/urdf/inc/solid3_property.xacro (robot description, xacro)
@@ -2,5 +2,5 @@
 <robot xmlns:xacro="http://ros.org/wiki/xacro">
   <xacro:macro name="solid3_property">
-     <xacro:property name="yaml_file" value="${xacro.load_yaml(/home/eliseev/workspace/urdf_expansion_ws/src/URDF_Expansion/config/input/solid3_property.xacro)}"/>
+     <xacro:property name="yaml_file" value="${xacro.load_yaml(/home/eliseev/workspace/urdf_expansion_ws/src/URDF_Expansion/config//solid3_description/solid3_property.xacro)}"/>
    <!-- TODO -->
    <!-- <xacro:property name="yaml_path" value="$(find generate_robot_urdf)/config/output/joint_limits.yaml" /> -->

File: config/solid3_description/urdf/solid3_macro.xacro (robot description, xacro)
@@ -2,5 +2,5 @@
 <robot xmlns:xacro="http://ros.org/wiki/xacro">
  <xacro:macro name="solid3" params="parent_link">
-<xacro:include filename="$(find /home/eliseev/workspace/urdf_expansion_ws/src/URDF_Expansion/config/input/solid3_macro.xacro" />
+<xacro:include filename="$(find /home/eliseev/workspace/urdf_expansion_ws/src/URDF_Expansion/config//solid3_description/solid3_macro.xacro" />
   <!-- TODO -->
   <!-- <xacro:include filename="$(find ur_description)/urdf/inc/ur_common.xacro" /> -->/n
